Commit message: Everything Works just sligght offset for ball placing

File: src/kortex_description/grippers/gen3_lite_2f/urdf/gen3_lite_2f_macro.xacro (robot description, xacro)
@@ -65,8 +65,9 @@
           </material>
         </visual>
-        <collision>
-          <origin xyz="0 0 0" rpy="0 0 0" />
-          <geometry>
-            <mesh filename="file://$(find kortex_description)/grippers/gen3_lite_2f/meshes/gripper_base_link.STL" />
+        <!-- Primitive collision for dartsim compatibility (mesh collisions not supported) -->
+        <collision>
+          <origin xyz="0 0 0.04" rpy="0 0 0" />
+          <geometry>
+            <cylinder radius="0.025" length="0.08" />
           </geometry>
         </collision>
@@ -90,8 +91,9 @@
         </material>
       </visual>
+      <!-- Primitive box collision for dartsim compatibility -->
       <collision>
-        <origin xyz="0 0 0" rpy="0 0 0" />
-        <geometry>
-          <mesh filename="file://$(find kortex_description)/grippers/gen3_lite_2f/meshes/right_finger_prox_link.STL" />
+        <origin xyz="0.022 0.005 0" rpy="0 0 0" />
+        <geometry>
+          <box size="0.050 0.018 0.024" />
         </geometry>
       </collision>
@@ -99,4 +101,9 @@
       <gazebo reference="${prefix}right_finger_prox_link">
         <material>Kortex/Gray</material>
+        <mu1>2.5</mu1>
+        <mu2>2.5</mu2>
+        <kp>1000000</kp>
+        <kd>100</kd>
+        <minDepth>0.001</minDepth>
       </gazebo>
       <joint name="${prefix}right_finger_bottom_joint" type="revolute">
@@ -123,8 +130,9 @@
           </material>
         </visual>
-        <collision>
-          <origin xyz="0 0 0" rpy="0 0 0" />
-          <geometry>
-            <mesh filename="file://$(find kortex_description)/grippers/gen3_lite_2f/meshes/right_finger_dist_link.STL" />
+        <!-- Primitive box collision for dartsim compatibility -->
+        <collision>
+          <origin xyz="0.018 0.001 0" rpy="0 0 0" />
+          <geometry>
+            <box size="0.044 0.016 0.024" />
           </geometry>
         </collision>
@@ -132,4 +140,9 @@
       <gazebo reference="${prefix}right_finger_dist_link">
         <material>Kortex/Blue</material>
+        <mu1>2.5</mu1>
+        <mu2>2.5</mu2>
+        <kp>1000000</kp>
+        <kd>100</kd>
+        <minDepth>0.001</minDepth>
       </gazebo>
       <joint name="${prefix}right_finger_tip_joint" type="revolute">
@@ -156,8 +169,9 @@
           </material>
         </visual>
-        <collision>
-          <origin xyz="0 0 0" rpy="0 0 0" />
-          <geometry>
-            <mesh filename="file://$(find kortex_description)/grippers/gen3_lite_2f/meshes/left_finger_prox_link.STL" />
+        <!-- Primitive box collision for dartsim compatibility -->
+        <collision>
+          <origin xyz="0.022 0.005 0" rpy="0 0 0" />
+          <geometry>
+            <box size="0.050 0.018 0.024" />
           </geometry>
         </collision>
@@ -165,4 +179,9 @@
       <gazebo reference="${prefix}left_finger_prox_link">
         <material>Kortex/Gray</material>
+        <mu1>2.5</mu1>
+        <mu2>2.5</mu2>
+        <kp>1000000</kp>
+        <kd>100</kd>
+        <minDepth>0.001</minDepth>
       </gazebo>
       <joint name="${prefix}left_finger_bottom_joint" type="revolute">
@@ -190,8 +209,9 @@
           </material>
         </visual>
-        <collision>
-          <origin xyz="0 0 0" rpy="0 0 0" />
-          <geometry>
-            <mesh filename="file://$(find kortex_description)/grippers/gen3_lite_2f/meshes/left_finger_dist_link.STL" />
+        <!-- Primitive box collision for dartsim compatibility -->
+        <collision>
+          <origin xyz="-0.018 0.001 0" rpy="0 0 0" />
+          <geometry>
+            <box size="0.044 0.016 0.024" />
           </geometry>
         </collision>
@@ -199,4 +219,9 @@
       <gazebo reference="${prefix}left_finger_dist_link">
         <material>Kortex/Blue</material>
+        <mu1>2.5</mu1>
+        <mu2>2.5</mu2>
+        <kp>1000000</kp>
+        <kd>100</kd>
+        <minDepth>0.001</minDepth>
       </gazebo>
       <joint name="${prefix}left_finger_tip_joint" type="revolute">
